File: kicad/current_version/working/working.kicad_sch (KiCad schematic)
At the start: 4 parts, among them IC1 imsp10mpump21rs2227

Commit message: first works
Parts:
- removed C1: c6nf100, oomlout_oomp_part_footprints:c6nf100_electronic_capacitor_0603_100_nano_farad, symbol oomlout_oomp_part_symbols:c6nf100_electronic_capacitor_0603_100_nano_farad
- removed IC1: imsp10mpump21rs2227, oomlout_oomp_part_footprints:imsp10mpump21rs2227_electronic_ic_msop_10_multiplexer_usb_multiplexer_two_to_one_jiangsu_r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, symbol oomlout_oomp_part_symbols:imsp10mpump21rs2227_electronic_ic_msop_10_multiplexer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
- removed R1, R2: r6o103, oomlout_oomp_part_footprints:r6o103_electronic_resistor_0603_10000_ohm, symbol oomlout_oomp_part_symbols:r6o103_electronic_resistor_0603_10000_ohm
- added BB_MEGA_1: bbmcu_electronic_breakout_board_pico_mcu_raspberr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, oomlout_oomp_part_footprints:bbmcu_electronic_breakout_board_pico_mcu_raspberry_pi_2040, symbol oomlout_oomp_part_symbols:bbmcu_electronic_breakout_board_pico_mcu_raspberry_pi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
- added BB_MEGA_2: bbmcu_electronic_breakout_board_shennie_mcu_atmeg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, oomlout_oomp_part_footprints:bbmcu_electronic_breakout_board_shennie_mcu_atmega328p_arduino_compatible, symbol oomlout_oomp_part_symbols:bbmcu_electronic_breakout_board_shennie_mcu_atmega328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
- added BB_MEGA_3: bbmcu_electronic_breakout_board_devkitc_mcu_espre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, oomlout_oomp_part_footprints:bbmcu_electronic_breakout_board_devkitc_mcu_espressif_esp32, symbol oomlout_oomp_part_symbols:bbmcu_electronic_breakout_board_devkitc_mcu_espressif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
- added J1, J2: hob3thra, oomlout_oomp_part_footprints:hob3thra_electronic_header_oobb_i2c_triple_through_hole_right_angle, symbol oomlout_oomp_part_symbols:hob3thra_electronic_header_oobb_i2c_triple_through_ho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
- added J10, J3, J4, J5, J6, J7, J8, J9: hob3thra, oomlout_oomp_part_footprints:hob3thra_electronic_header_oobb_basic_triple_through_hole_right_angle, symbol oomlout_oomp_part_symbols:hob3thra_electronic_header_oobb_basic_triple_through_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
Connections:
- net +5V: now also BB_MEGA_1.40 (___vbus), BB_MEGA_2.27 (+5V), BB_MEGA_3.19 (___5v)
- net GND: now also BB_MEGA_1.13 (___gnd), BB_MEGA_1.18 (___gnd), BB_MEGA_1.23 (___gnd), BB_MEGA_1.28 (___gnd), BB_MEGA_1.3 (___gnd), BB_MEGA_1.33 (___gnd_adc), BB_MEGA_1.38 (___gnd), BB_MEGA_1.8 (___gnd), BB_MEGA_2.29 (GND), BB_MEGA_2.4 (GND), BB_MEGA_3.14 (___gnd), BB_MEGA_3.32 (___gnd), BB_MEGA_3.38 (___gnd), J1.1 (gnd), J10.1 (gnd), J2.1 (gnd), J3.1 (gnd), J4.1 (gnd), J5.1 (gnd), J6.1 (gnd), J7.1 (gnd), J8.1 (gnd), J9.1 (gnd)
- new net +3V3: BB_MEGA_2.17 (3V3), BB_MEGA_3.1 (___3v3)
- new net 3v3_enable_mbyy: BB_MEGA_1.37 (___3v3_enable)
- new net 3v3_out_mbyy: BB_MEGA_1.36 (___3v3_out)
- new net a0_mbyy: BB_MEGA_1.31 (___a0), BB_MEGA_2.19 (A0)
- new net a1_mbyy: BB_MEGA_1.32 (___a1), BB_MEGA_2.20 (A1)
- new net a2_mbyy: BB_MEGA_1.34 (___a2), BB_MEGA_2.21 (A2)
- new net a3_mbyy: BB_MEGA_2.22 (A3)
- new net a4_mbyy: BB_MEGA_2.23 (A4)
- new net a5_mbyy: BB_MEGA_2.24 (A5)
- new net a6_mbyy: BB_MEGA_2.25 (A6)
- new net a7_mbyy: BB_MEGA_2.26 (A7)
- new net aref_mbyy: BB_MEGA_2.18 (AREF)
- new net d0_mbyy: BB_MEGA_1.1 (___gp0), BB_MEGA_2.2 (D0/RX), BB_MEGA_3.34 (___rx), J1.3 (sda), J2.3 (sda), J3.3 (data_1)
- new net d0_nnn: BB_MEGA_1.5 (___gp3), BB_MEGA_2.6 (D3), BB_MEGA_3.6 (___io35), J8.3 (data_1)
- new net d0_ooo: BB_MEGA_1.9 (___gp6), BB_MEGA_2.9 (D6), BB_MEGA_3.9 (___io25), J4.3 (data_1)
- new net d0_ppp: BB_MEGA_1.12 (___gp9), BB_MEGA_2.12 (D9), BB_MEGA_3.12 (___io14), J7.3 (data_1)
- new net d0_qqq: BB_MEGA_1.16 (___gp12), BB_MEGA_2.15 (D12), BB_MEGA_3.23 (___io15), J6.3 (data_1)
- new net d0_rrr: BB_MEGA_1.20 (___gp15), BB_MEGA_3.26 (___io4), J5.3 (data_1)
- new net d0_sss: BB_MEGA_1.24 (___gp18), BB_MEGA_3.29 (___io5)
- new net d0_ttt: BB_MEGA_1.27 (___gp21), BB_MEGA_3.33 (___io21), J9.3 (data_1)
- new net d0_zz: J10.3 (data_1)
- new net d10_mbyy: BB_MEGA_1.14 (___gp10), BB_MEGA_2.13 (D10), BB_MEGA_3.13 (___io12), J7.4 (data_3)
- new net d11_mbyy: BB_MEGA_1.15 (___gp11), BB_MEGA_2.14 (D11), BB_MEGA_3.15 (___io13), J7.4 (data_3)
- new net d13_mbyy: BB_MEGA_1.17 (___gp13), BB_MEGA_2.16 (D13), BB_MEGA_3.24 (___io2), J6.4 (data_3)
- new net d14_mbyy: BB_MEGA_1.19 (___gp14), BB_MEGA_3.25 (___io0), J6.4 (data_3)
- new net d16_mbyy: BB_MEGA_1.21 (___gp16), BB_MEGA_3.27 (___io16), J5.4 (data_3)
- new net d17_mbyy: BB_MEGA_1.22 (___gp17), BB_MEGA_3.28 (___io17), J5.4 (data_3)
- new net d19_mbyy: BB_MEGA_1.25 (___gp19), BB_MEGA_3.30 (___io18)
- new net d1_mbyy: BB_MEGA_1.2 (___gp1), BB_MEGA_2.1 (D1/TX), BB_MEGA_3.35 (___tx), J3.4 (data_3)
- new net d1_nnn: BB_MEGA_1.6 (___gp4), BB_MEGA_2.7 (D4), BB_MEGA_3.7 (___io32), J8.4 (data_3)
- new net d1_ooo: BB_MEGA_1.10 (___gp7), BB_MEGA_2.10 (D7), BB_MEGA_3.10 (___io26), J4.4 (data_3)
- new net d1_ttt: BB_MEGA_1.29 (___gp22), BB_MEGA_3.36 (___io22), J9.4 (data_3)
- new net d1_zz: J10.4 (data_3)
- new net d20_mbyy: BB_MEGA_1.26 (___gp20), BB_MEGA_3.31 (___io19)
- new net d23_mbyy: BB_MEGA_3.37 (___io23), J9.4 (data_3)
- new net d2_mbyy: BB_MEGA_1.4 (___gp2), BB_MEGA_2.5 (D2), BB_MEGA_3.5 (___io34), J1.4 (scl), J2.4 (scl), J3.4 (data_3)
- new net d2_nnn: BB_MEGA_1.7 (___gp5), BB_MEGA_2.8 (D5), BB_MEGA_3.8 (___io33), J8.4 (data_3)
- new net d2_ooo: BB_MEGA_1.11 (___gp8), BB_MEGA_2.11 (D8), BB_MEGA_3.11 (___io27), J4.4 (data_3)
- new net d2_zz: J10.4 (data_3)
- new net ref_mbyy: BB_MEGA_1.35 (___vref)
- new net reset_mbyy: BB_MEGA_2.28 (~{RESET}), BB_MEGA_2.3 (~{RESET}), BB_MEGA_3.2 (___enable)
- new net run_mbyy: BB_MEGA_1.30 (___run)
- new net vin_mbyy: BB_MEGA_2.30 (VIN)
- new net vmcu: J1.2 (power), J10.2 (power), J2.2 (power), J3.2 (power), J4.2 (power), J5.2 (power), J6.2 (power), J7.2 (power), J8.2 (power), J9.2 (power)
- new net vsys_mbyy: BB_MEGA_1.39 (___vsys)
Other:
- note added: "aaa"
- note added: "bbb"
- note added: "breakout_board_mcu_devkitc_esp32"
- note added: "breakout_board_mcu_nano_atmega328p_arduino_compatible"
- note added: "breakout_board_mcu_pico_raspberry_pi_2040"
- note added: "connector_oobb_basic_through_hole_triple"
- note added: "connector_oobb_i2c_through_hole_triple"
- note added: "digital_pins"
- note added: "esp32"
- note added: "glue"
- note added: "i2c_pins"
- note added: "logic_glue"
- note added: "mbyy"
- note added: "mmm"
- note added: "nano"
- note added: "nnn"
- note added: "oobb_basic_triple"
- note added: "oobb_i2c_triple"
- note added: "oomlout_oomp_electronic_project_mcu_breakout_mega_footprint"
- note added: "oomp breakout_board mcu devkitc esp32"
- note added: "oomp breakout_board mcu nano atmega328p arduino_compatible"
- note added: "oomp breakout_board mcu pico raspberry_pi_2040"
- note added: "oomp connector oobb_basic through_hole triple"
- note added: "oomp connector oobb_i2c through_hole triple"
- note added: "oomp logic glue"
- note added: "ooo"
- note added: "pi_pico"
- note added: "ppp"
- note added: "qqq"
- note added: "rrr"
- note added: "ttt"
- note removed: "ic_usb_multiplexer_msop_10_two_to_one_rs2227xn"
- note removed: "oomp ic usb_multiplexer msop_10 two_to_one rs2227xn"
- note removed: "oomp_"
- note removed: "usb_multi_rs2227"
